File: Gerbers 3/MRCS-Tiny85-Servo-Auto.brd (EAGLE design)
At the start: 48.3 x 48.3 mm, 18 parts, among them U1 ATTINY85-20PU

Commit message: Moved one of the push buttons away from socket
This makes it easier to remove the ATTiny for reprogramming
Parts:
- moved S1 10.2 mm to (24.1, 6.35)
Routing:
- net INPUT: track 56.5 -> 40.1 mm
Other:
- board text added: "20220828 v1.1"
- board text removed: "20221007 v1.2"
Changed lines of the file:
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@@
 <hole x="3.81" y="44.45" drill="2.794"/>
 <text x="1.905" y="0.635" size="1.6764" layer="51" font="vector">ATTiny85 Auto Servo</text>
-<text x="31.115" y="1.27" size="1.4224" layer="21" font="vector">20221007 v1.2</text>
+<text x="31.115" y="1.27" size="1.4224" layer="21" font="vector">20220828 v1.1</text>
 <text x="45.72" y="41.275" size="1.6764" layer="22" font="vector" rot="MR0">Seth Neumann, Lawrence Crowl</text>
 <text x="42.545" y="8.255" size="1.6764" layer="21" font="vector">GND
@@
 <attribute name="VALUE" x="12.192" y="37.973" size="1.27" layer="21" ratio="15" rot="R180"/>
 </element>
-<element name="S1" library="SparkFun-Electromechanical" package="TACTILE-PTH" value="" x="34.29" y="6.35" smashed="yes">
-<attribute name="NAME" x="31.75" y="10.16" size="1.27" layer="25" ratio="10"/>
+<element name="S1" library="SparkFun-Electromechanical" package="TACTILE-PTH" value="" x="24.13" y="6.35" smashed="yes">
+<attribute name="NAME" x="21.59" y="10.16" size="1.27" layer="25" ratio="10"/>
 </element>
 <element name="U1" library="ATTINY85-20PU" package="DIP762W46P254L927H533Q8B" value="ATTINY85-20PU" x="24.13" y="17.78" smashed="yes">
@@
 <wire x1="27.94" y1="19.05" x2="27.94" y2="19.685" width="0.3048" layer="16"/>
 <wire x1="40.767" y1="24.13" x2="32.385" y2="24.13" width="0.3048" layer="16"/>
+<wire x1="27.94" y1="19.05" x2="30.48" y2="16.51" width="0.3048" layer="1"/>
+<wire x1="30.48" y1="16.51" x2="30.48" y2="11.43" width="0.3048" layer="1"/>
+<wire x1="30.48" y1="11.43" x2="27.6606" y2="8.6106" width="0.3048" layer="1"/>
 <contactref element="S1" pad="1"/>
 <contactref element="S1" pad="2"/>
 <contactref element="C2" pad="1"/>
 <contactref element="J1" pad="7"/>
-<wire x1="31.0388" y1="8.6106" x2="15.320390625" y2="8.6106" width="0.3048" layer="16"/>
+<wire x1="20.8788" y1="8.6106" x2="15.320390625" y2="8.6106" width="0.3048" layer="16"/>
 <wire x1="15.320390625" y1="8.6106" x2="15.24" y2="8.5725" width="0.3048" layer="16"/>
-<wire x1="31.0388" y1="8.6106" x2="37.5412" y2="8.6106" width="0.3048" layer="16"/>
-<wire x1="27.94" y1="19.05" x2="35.56" y2="19.05" width="0.4064" layer="1"/>
-<wire x1="35.56" y1="19.05" x2="37.465" y2="17.145" width="0.4064" layer="1"/>
-<wire x1="37.465" y1="17.145" x2="37.465" y2="8.6868" width="0.4064" layer="1"/>
-<wire x1="37.465" y1="8.6868" x2="37.5412" y2="8.6106" width="0.4064" layer="1"/>
+<wire x1="20.8788" y1="8.6106" x2="27.3812" y2="8.6106" width="0.3048" layer="16"/>
 <wire x1="40.767" y1="24.13" x2="40.513" y2="24.13" width="0" layer="19" extent="16-16"/>
+<wire x1="27.3812" y1="8.6106" x2="27.6606" y2="8.6106" width="0" layer="19" extent="1-1"/>
 </signal>
 <signal name="SERVO">
